File: hardware/rp2040-mgmt-module/rp2040-mgmt-module.kicad_pcb (KiCad board)
At the start: 2 copper layers, 77 x 24 mm, 86 parts, among them J1 SWD, J2 Bus_PCI_Express_x1, J3 USB_B_Micro, J4 RJ45_Hanrun_HR913550A_Horizon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, J5 ADC, J6 UART, J7 UART, SW1 BOOT, SW2 RESET, U1 W5500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

Commit message: feat: add pcb labels
Parts:
- moved R23 3.85 mm to (104.5, 65.8)
- moved R24 2.20 mm to (103.4, 65.8)
Routing:
- net /ADC_AVDD: track 5.28 -> 7.92 mm
Other:
- board text added: "BOOT"
- board text added: "GP10"
- board text added: "GP11"
- board text added: "GP27"
- board text added: "GP28"
- board text added: "GP8"
- board text added: "GP9"
- board text added: "RESET"
- board text added: "SWCLK"
- board text added: "SWDIO"
