File: hardware/esp32-mgmt-module/esp32-mgmt-module.kicad_sch (KiCad schematic)
At the start: 89 parts, among them J1 Bus_PCI_Express_x1, J2 BOOT, J3 RJ45_Hanrun_HR913550A_Horizon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, J4 GPIO, J5 SWD, J6 USB_C, J7 UART, Q1 MMBT3904, Q2 MMBT3904, SW1 RESET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

Commit message: fix: add component placement corrections
Parts:
- SW1: JLCPCB_CORRECTION (none) -> 0;2.4;180
- U2: JLCPCB_CORRECTION (none) -> 0;0;180
Changed lines of the file:
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@@
 			)
 		)
+		(property "JLCPCB_CORRECTION" "0;0;180"
+			(at 95.25 261.62 0)
+			(effects
+				(font
+					(size 1.27 1.27)
+				)
+				(hide yes)
+			)
+		)
 		(pin "2"
 		)
@@
 			(at 110.49 121.92 0)
 			(effects
+				(font
+					(size 1.27 1.27)
+				)
+				(hide yes)
+			)
+		)
+		(property "JLCPCB_CORRECTION" "0;2.4;180"
+			(at 110.49 121.92 0)
+			(effects
