File: hardware/esp32-mgmt-module/esp32-mgmt-module.kicad_pcb (KiCad board)
At the start: 4 copper layers, 77 x 31.8 mm, 91 parts, among them J1 Bus_PCI_Express_x1, J2 BOOT, J3 RJ45_Hanrun_HR913550A_Horizon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, J4 GPIO, J5 SWD, J6 USB_C, J7 UART, Q1 MMBT3904, Q2 MMBT3904, SW1 RESET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

Commit message: feat: add status led
fix: switch swdio from input-only pins
Parts:
- added D2: BLUE LED, LED_SMD:LED_0603_1608Metric, F.Cu at (81.3, 53.5)
- added R36: 470R, Resistor_SMD:R_0402_1005Metric, F.Cu at (82.7, 53.5)
- D4: value RED -> RED LED
Connections:
- C11 pad 1: /~{RESET} -> /~{I2C_RESET}
- Q2 pad 3: /~{RESET} -> /~{I2C_RESET}
- R16 pad 1: /~{RESET} -> /~{I2C_RESET}
- SW1 pad 2: /~{RESET} -> /~{I2C_RESET}
- U4 pad 24: /SW_A0 -> /STATUS_LED
- U4 pad 3: /~{RESET} -> /~{I2C_RESET}
- U4 pad 4: /~{ALERT} -> /SWCLK
- U4 pad 5: /OVERLOAD -> /SWDIO
- U4 pad 6: /SWDIO -> /~{ALERT}
- U4 pad 8: /~{I2C_RESET} -> /SW_A0
- U4 pad 9: /SWCLK -> /OVERLOAD
Routing:
- net /~{I2C_RESET}: track 41.1 -> 91.5 mm, vias 2 -> 4
- net /~{RESET}: track 47.1 -> 0.00 mm, vias 2 -> 0
- net /SW_A0: track 26.8 -> 41.7 mm
- net /SWCLK: track 44.8 -> 40.7 mm
- net /OVERLOAD: track 41.6 -> 45.5 mm
- net /STATUS_LED: track 0.00 -> 2.70 mm
- net Net-(D2-A): track 0.00 -> 1.94 mm
- net /~{ALERT}: track 39.6 -> 41.0 mm
- net /SWDIO: track 42.3 -> 41.6 mm
