File: hardware/controller/controller.kicad_sch (KiCad schematic)
At the start: 82 parts, among them J1 Bus_PCI_Express_x1, J2 USB, J4 BM03B-SRSS-TB(LF)(SN), J6 RJ45_Hanrun_HR913550A_Horizon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, SW1 434133025816, SW2 434133025816, U1 RP2350A, U2 NCP1117ST33T3G, U3 W25Q128JVSIQ, U4 W6100-L, U5 RPi Radio Module 2, X1 12MHz, Y2 X322525MRB4SI

Commit message: chore(controller): clean up production settings
Parts:
- J4, L1, U2: JLCPCB_CORRECTION (none) -> 0;0;180
- U1: JLCPCB_CORRECTION (none) -> 0;0;0
- U3, U4: JLCPCB_CORRECTION (none) -> 0;0;270
- U5: LCSC (none) -> C49451547
Other:
- note removed: "If using RP2354 (internal flash), remove R10. R9 can be fit to use U3 as secondary memory."
Changed lines of the file:
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@@
 		)
 	)
-	(text "If using RP2354 (internal flash), remove R10.\nR9 can be fit to use U3 as secondary memory."
-		(exclude_from_sim no)
-		(at 35.306 111.506 0)
-		(effects
-			(font
-				(size 1.27 1.27)
-			)
-			(justify left bottom)
-		)
-	)
 	(text "Power"
 		(exclude_from_sim no)
@@
 			)
 		)
+		(property "JLCPCB_CORRECTION" "0;0;180"
+			(at 246.38 110.49 0)
+			(hide yes)
+			(show_name no)
+			(do_not_autoplace no)
+			(effects
+				(font
+					(size 1.27 1.27)
+				)
+			)
+		)
 		(pin "1"
 		)
@@
 			)
 		)
+		(property "JLCPCB_CORRECTION" "0;0;180"
+			(at 365.76 212.09 0)
+			(hide yes)
+			(show_name no)
+			(do_not_autoplace no)
+			(effects
+				(font
+					(size 1.27 1.27)
+				)
+			)
+		)
 		(pin "1"
 		)
@@
 			)
 		)
+		(property "JLCPCB_CORRECTION" "0;0;0"
+			(at 229.87 162.56 0)
+			(hide yes)
+			(show_name no)
+			(do_not_autoplace no)
+			(effects
+				(font
+					(size 1.27 1.27)
+				)
+			)
+		)
 		(pin "1"
 		)
@@
 			)
 		)
+		(property "LCSC" " C49451547"
+			(at 373.38 104.14 0)
+			(hide yes)
+			(show_name no)
+			(do_not_autoplace no)
+			(effects
+				(font
+					(size 1.27 1.27)
+				)
+			)
+		)
 		(pin "21"
 		)
@@
 			)
 		)
+		(property "JLCPCB_CORRECTION" "0;0;270"
+			(at 91.44 144.78 0)
+			(hide yes)
+			(show_name no)
+			(do_not_autoplace no)
+			(effects
+				(font
+					(size 1.27 1.27)
+				)
+			)
+		)
 		(pin "1"
 		)
@@
 			)
 		)
+		(property "JLCPCB_CORRECTION" "0;0;270"
+			(at 114.3 346.71 0)
+			(hide yes)
+			(show_name no)
+			(do_not_autoplace no)
+			(effects
+				(font
+					(size 1.27 1.27)
+				)
+			)
+		)
 		(pin "43"
 		)
@@
 			(at 177.8 48.26 0)
 			(hide yes)
+			(show_name no)
+			(do_not_autoplace no)
+			(effects
+				(font
+					(size 1.27 1.27)
+				)
+			)
+		)
+		(property "JLCPCB_CORRECTION" "0;0;180"
+			(at 177.8 48.26 0)
+			(hide yes)

Commit message: feat(controller): add RPi RM2 and wire up remaining pins
fix(controller): move rj45 jack inset 1mm
Parts:
- removed D1, D2: 1N5819WS, Diode_SMD:D_SOD-323, symbol Device:D_Schottky
- removed U2: NCP1117ST33T3G, Package_TO_SOT_SMD:SOT-223, symbol RPI_DB:Integrated_Circuits | Power | LDO/RP-01JWD9-7JRX6J
- added C18, C27: 100nF, Capacitor_SMD:C_0402_1005Metric, symbol Device:C
- added Q1, Q2: 2N7002, Package_TO_SOT_SMD:SOT-23, symbol Transistor_FET:2N7002
- added R10, R11: 100K, Local Library:R_0402_1005Metric, symbol Device:R
- added R12: 0R, Local Library:R_0603_1608Metric, symbol Device:R
- added R13: 120K, Local Library:R_0603_1608Metric, symbol Device:R
- added R14: 10K, Local Library:R_0402_1005Metric, symbol Device:R
- added R15: 1K, Local Library:R_0402_1005Metric, symbol Device:R
- added R32, R41, R43: 4.7K, Local Library:R_0402_1005Metric, symbol Device:R
- added SW3: SW_Push, Button_Switch_SMD:SW_SPST_B3U-3000P, symbol Switch:SW_Push
- added U2: AP7361C-33E, Package_TO_SOT_SMD:SOT-223-3_TabPin2, symbol Regulator_Linear:AP7361C-33E
- J1: now fitted; now in the parts list
Connections:
- net GPIO29_ADC3 is gone; now on net GPIO29: U1.43 (GPIO29_ADC3)
- net SCL is gone; now on net GPIO5: J1.A14 (SCL)
- net SDA is gone; now on net GPIO4: J1.B14 (SDA)
- net ~{ALERT} is gone; now on net GPIO7: J1.B15 (~{ALERT})
- net +3.3V: now also R32.2, R41.2, R43.2, U2.3 (VO)
- net +5V: now also J1.A12 (+5V), J1.B12 (+5V), R12.2, U2.1 (VI)
- net GND: now also J1.A1 (GND), J1.B17 (GND), C18.2, C27.2, Q1.2 (S), Q2.2 (S), R10.2, R11.2, R14.2, SW3.2, U2.2 (GND); no longer J1.A15 (GND), J1.B10 (GND), J1.B9 (PGND)
- net GPIO2: now also J1.B10 (LED_DATA)
- net GPIO20: now also R25.2, U4.48 (~{RST}); no longer U4.47 (~{INT})
- net GPIO21: now also U4.47 (~{INT}); no longer R25.2, U4.48 (~{RST})
- net GPIO28_ADC2: now also C18.1, R13.2, R14.1
- net GPIO4: now also R32.1
- net GPIO5: now also R41.1
- net GPIO6: now also J1.A15 (~{EXP_INT})
- net GPIO7: now also R43.1
- net GPIO8: now also Q2.1 (G), R11.1
- net VIN: now also R13.1
- net at J2.1 (Pin_1): now also R12.1
- net EN renamed ~{MUX_RST}
- net ~{MUX_RST}: now also Q2.3 (D)
- net GPIO1 renamed EXP_RST_GATE
- net EXP_RST_GATE: now also Q1.1 (G), R10.1
- net GPIO22 renamed BUTTON
- net BUTTON: now also C27.1, R15.1
- new net: R15.2, SW3.1
- new net ~{EXP_RST}: J1.B9 (~{EXP_RST}), Q1.3 (D)
