File: hardware/controller/controller.kicad_sch (KiCad schematic)
At the start: 97 parts, among them J1 Bus_PCI_Express_x1, J2 USB, J4 BM03B-SRSS-TB(LF)(SN), J5 BM03B-SRSS-TB(LF)(SN), J6 RJ45_Hanrun_HR913550A_Horizon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, Q1 2N7002, Q2 2N7002, SW1 434133025816, SW2 434133025816, SW3 SW_Push, U1 RP2350A, U2 AP7361C-33E, U3 W25Q128JVSIQ, U4 W6100-L, U5 RPi Radio Module 2, X1 12MHz, Y2 X322525MRB4SI

Commit message: fix(controller): correct C6/C7 footprint name and assembly fields
- Rename Local Library C_0805_Wide to C_0402_Wide; its pads were always
  an 0402 land, matching the C23733 (CL05A475MP5NRNC) part it carries
- Drop stale RPI_DB manufacturer_pn/lcsc_pn fields from C6/C7/C9 that
  named a different part than the LCSC field
- Mark J1 card edge DNP and out of the BOM/position files
- Add 180 degree JLCPCB rotation correction for Q1/Q2

Co-Authored-By: Claude Opus 5.5 <noreply@anthropic.com>
Parts:
- C6, C7: footprint Local Library:C_0805_Wide -> Local Library:C_0402_Wide; manufacturer_pn GRM155R60J475ME47D -> (none)
- C9: manufacturer_pn GRM155R60J475ME47D -> (none)
- J1: now not fitted; now left out of the parts list
- Q1, Q2: JLCPCB_CORRECTION (none) -> 0;0;180
Changed lines of the file:
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@@
 		(body_style 1)
 		(exclude_from_sim no)
-		(in_bom yes)
+		(in_bom no)
 		(on_board yes)
-		(in_pos_files yes)
-		(dnp no)
+		(in_pos_files no)
+		(dnp yes)
 		(fields_autoplaced yes)
 		(property "Reference" "J1"
@@
 			)
 		)
+		(property "JLCPCB_CORRECTION" "0;0;180"
+			(at 349.25 165.1 0)
+			(hide yes)
+			(show_name no)
+			(do_not_autoplace no)
+			(effects
+				(font
+					(size 1.27 1.27)
+				)
+			)
+		)
 		(pin "3"
 		)
@@
 			)
 		)
-		(property "Footprint" "Local Library:C_0805_Wide"
+		(property "Footprint" "Local Library:C_0402_Wide"
 			(at 266.7 110.49 0)
 			(hide yes)
@@
 			)
 		)
-		(property "manufacturer_pn" "GRM155R60J475ME47D"
-			(at 266.7 110.49 0)
-			(hide yes)
-			(show_name no)
-			(do_not_autoplace no)
-			(effects
-				(font
-					(size 1.27 1.27)
-				)
-			)
-		)
 		(property "packaging" "180mm paper taping"
 			(at 266.7 110.49 0)
@@
 			)
 		)
+		(property "JLCPCB_CORRECTION" "0;0;180"
+			(at 389.89 165.1 0)
+			(hide yes)
+			(show_name no)
+			(do_not_autoplace no)
+			(effects
+				(font
+					(size 1.27 1.27)
+				)
+			)
+		)
 		(pin "3"
 		)
@@
 			)
 		)
-		(property "Footprint" "Local Library:C_0805_Wide"
+		(property "Footprint" "Local Library:C_0402_Wide"
 			(at 255.27 110.49 0)
 			(hide yes)
@@
 			)
 		)
-		(property "manufacturer_pn" "GRM155R60J475ME47D"
-			(at 255.27 110.49 0)
-			(hide yes)
-			(show_name no)
-			(do_not_autoplace no)
-			(effects
-				(font
-					(size 1.27 1.27)
-				)
-			)
-		)
 		(property "packaging" "180mm paper taping"
 			(at 255.27 110.49 0)
@@
 			(at 293.37 133.35 0)
 			(hide yes)
-			(show_name no)
-			(do_not_autoplace no)
-			(effects
-				(font
-					(size 1.27 1.27)
-				)
-			)
-		)
-		(property "manufacturer_pn" "GRM155R60J475ME47D"
-			(at 293.37 133.35 0)
-			(hide yes)
