File: hardware/controller/controller.kicad_pcb (KiCad board)
At the start: 4 copper layers, 92.8 x 28 mm, 97 parts, among them J1 Bus_PCI_Express_x1, J2 USB, J4 BM03B-SRSS-TB(LF)(SN), J5 BM03B-SRSS-TB(LF)(SN), J6 RJ45_Hanrun_HR913550A_Horizon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, Q1 2N7002, Q2 2N7002, SW1 434133025816, SW2 434133025816, SW3 SW_Push, U1 RP2350A, U2 AP7361C-33E, U3 W25Q128JVSIQ, U4 W6100-L, U5 RPi Radio Module 2, X1 12MHz, Y2 X322525MRB4SI

Commit message: fix(controller): correct C6/C7 footprint name and assembly fields
- Rename Local Library C_0805_Wide to C_0402_Wide; its pads were always
  an 0402 land, matching the C23733 (CL05A475MP5NRNC) part it carries
- Drop stale RPI_DB manufacturer_pn/lcsc_pn fields from C6/C7/C9 that
  named a different part than the LCSC field
- Mark J1 card edge DNP and out of the BOM/position files
- Add 180 degree JLCPCB rotation correction for Q1/Q2

Co-Authored-By: Claude Opus 5.5 <noreply@anthropic.com>
Parts:
- C6, C7: footprint Local Library:C_0805_Wide -> Local Library:C_0402_Wide
Changed lines of the file:
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@@
 		)
 	)
-	(footprint "Local Library:C_0805_Wide"
+	(footprint "Local Library:C_0402_Wide"
 		(layer "F.Cu")
 		(at 110.35 59.05)
@@
 			)
 		)
-		(property "manufacturer_pn" "GRM155R60J475ME47D"
-			(at 0 0 0)
-			(unlocked yes)
-			(layer "F.Fab")
-			(hide yes)
-			(effects
-				(font
-					(size 1 1)
-					(thickness 0.15)
-				)
-			)
-		)
 		(property "packaging" "180mm paper taping"
 			(at 0 0 0)
@@
 			)
 		)
-		(property "lcsc_pn" "C82453"
-			(at 0 0 0)
-			(unlocked yes)
-			(layer "F.Fab")
-			(hide yes)
-			(effects
-				(font
-					(size 1 1)
-					(thickness 0.15)
-				)
-			)
-		)
 		(property "temp_coefficient" "X5R"
 			(at 0 0 0)
@@
 			)
 		)
-		(property "manufacturer_pn" "GRM155R60J475ME47D"
-			(at 0 0 90)
-			(unlocked yes)
-			(layer "F.Fab")
-			(hide yes)
-			(effects
-				(font
-					(size 1 1)
-					(thickness 0.15)
-				)
-			)
-		)
 		(property "packaging" "180mm paper taping"
 			(at 0 0 90)
@@
 		)
 	)
-	(footprint "Local Library:C_0805_Wide"
+	(footprint "Local Library:C_0402_Wide"
 		(layer "F.Cu")
 		(at 110.35 59.9)
@@
 			)
 		)
-		(property "manufacturer_pn" "GRM155R60J475ME47D"
-			(at 0 0 0)
-			(unlocked yes)
-			(layer "F.Fab")
-			(hide yes)
-			(effects
-				(font
-					(size 1 1)
-					(thickness 0.15)
-				)
-			)
-		)
 		(property "packaging" "180mm paper taping"
 			(at 0 0 0)
@@
 			)
 		)
-		(property "lcsc_pn" "C82453"
-			(at 0 0 0)
-			(unlocked yes)
-			(layer "F.Fab")
-			(hide yes)
-			(effects
-				(font
-					(size 1 1)
-					(thickness 0.15)
-				)
-			)
-		)
 		(property "temp_coefficient" "X5R"
 			(at 0 0 0)
@@
 			)
 		)
+		(attr exclude_from_pos_files exclude_from_bom dnp)
 		(duplicate_pad_numbers_are_jumpers no)
 		(fp_line
@@
 			(justify bottom)
 		)
-		(render_cache "Controller\nv0.3.2" 0
+		(render_cache "Controller\nv0.4.0" 0
 			(polygon
 				(pts
@@
 			(polygon
 				(pts
-					(xy 142.460154 56.424309) (xy 142.340536 56.416981) (xy 142.218811 56.397289) (xy 142.111833 56.370362)
-					(xy 142.03627 56.343342) (xy 142.097087 56.084964) (xy 142.236672 56.134331) (xy 142.327073 56.153361)
-					(xy 142.447606 56.160526) (xy 142.543037 56.153217) (xy 142.611465 56.13403) (xy 142.659548 56.105755)
-					(xy 142.696715 56.065224) (xy 142.718934 56.016901) (xy 142.726684 55.958293) (xy 142.720303 55.904593)
-					(xy 142.702504 55.862489) (xy 142.674155 55.827399) (xy 142.636375 55.799291) (xy 142.591665 55.77913)
-					(xy 142.536724 55.765586) (xy 142.413992 55.75606) (xy 142.292267 55.75606) (xy 142.292267 55.504002)
-					(xy 142.430753 55.504002) (xy 142.519963 55.495575) (xy 142.561187 55.48408) (xy 142.596533 55.467274)
-					(xy 142.626637 55.443697) (xy 142.650022 55.412594) (xy 142.664645 55.374945) (xy 142.669989 55.325399)
-					(xy 142.665601 55.287387) (xy 142.653136 55.256065) (xy 142.633887 55.229082) (xy 142.61018 55.207704)
-					(xy 142.582266 55.191308) (xy 142.549364 55.179311) (xy 142.479022 55.169877) (xy 142.391151 55.176877)
-					(xy 142.312234 55.197172) (xy 142.238312 55.22796) (xy 142.17265 55.264308) (xy 142.061458 55.03588)
-					(xy 142.140135 54.992008) (xy 142.239786 54.950059) (xy 142.35629 54.918643) (xy 142.419293 54.909304)
-					(xy 142.487448 54.906095) (xy 142.610627 54.914256) (xy 142.708824 54.936595) (xy 142.795778 54.974361)
-					(xy 142.863063 55.022874) (xy 142.916171 55.083534) (xy 142.95328 55.153299) (xy 142.975155 55.230414)
-					(xy 142.982681 55.316331) (xy 142.977449 55.372527) (xy 142.961603 55.427999) (xy 142.934412 55.483577)
-					(xy 142.898235 55.533542) (xy 142.855097 55.574277) (xy 142.804353 55.606584) (xy 142.875496 55.643084)
-					(xy 142.933332 55.688641) (xy 142.979567 55.743604) (xy 143.013369 55.80683) (xy 143.03421 55.878993)
-					(xy 143.041482 55.96214) (xy 143.032879 56.059702) (xy 143.007869 56.147246) (xy 142.965119 56.22583)
-					(xy 142.902997 56.293608) (xy 142.824255 56.347236) (xy 142.721463 56.389779) (xy 142.605619 56.415059)
+					(xy 142.957493 55.814678) (xy 143.112832 55.814678) (xy 143.112832 56.072599) (xy 142.957493 56.072599)
+					(xy 142.957493 56.395) (xy 142.651121 56.395) (xy 142.651121 56.072599) (xy 142.023631 56.072599)
+					(xy 142.023631 55.841973) (xy 142.038708 55.814678) (xy 142.321668 55.814678) (xy 142.651121 55.814678)
+					(xy 142.651121 55.323201) (xy 142.476915 55.556392) (xy 142.391341 55.684932) (xy 142.321668 55.814678)
+					(xy 142.038708 55.814678) (xy 142.139036 55.633053) (xy 142.293275 55.393726) (xy 142.472702 55.153391)
+					(xy 142.568637 55.039869) (xy 142.661563 54.941266) (xy 142.957493 54.941266)
 				)
 			)
@@
 			(polygon
 				(pts
-					(xy 144.729781 55.321461) (xy 144.72191 55.399559) (xy 144.698273 55.474601) (xy 144.662409 55.546224)
-					(xy 144.616482 55.616201) (xy 144.563294 55.682661) (xy 144.503093 55.747359) (xy 144.379353 55.866885)
-					(xy 144.311118 55.933014) (xy 144.240867 56.007478) (xy 144.181058 56.077728) (xy 144.158484 56.109614)
-					(xy 144.148544 56.131217) (xy 144.773927 56.131217) (xy 144.773927 56.395) (xy 143.804344 56.395)
-					(xy 143.800131 56.33629) (xy 143.800131 56.285915) (xy 143.808488 56.188094) (xy 143.832646 56.101267)
-					(xy 143.870262 56.020112) (xy 143.917734 55.944921) (xy 143.973467 55.875011) (xy 144.036253 55.809549)
-					(xy 144.167411 55.683612) (xy 144.261842 55.592295) (xy 144.339511 55.508398) (xy 144.369974 55.466619)
-					(xy 144.391993 55.426516) (xy 144.406226 55.384957) (xy 144.41086 55.343626) (xy 144.404144 55.284556)
-					(xy 144.386219 55.242732) (xy 144.358379 55.213566) (xy 144.301107 55.18564) (xy 144.228228 55.175739)
-					(xy 144.172948 55.180286) (xy 144.122257 55.193599) (xy 144.03204 55.23564) (xy 143.961698 55.283908)
-					(xy 143.917643 55.322651) (xy 143.762396 55.103382) (xy 143.861472 55.025472) (xy 143.977452 54.961691)
-					(xy 144.060864 54.930933) (xy 144.148358 54.912377) (xy 144.240867 54.906095) (xy 144.363903 54.913989)
-					(xy 144.461144 54.935496) (xy 144.547135 54.971833) (xy 144.613277 55.018294) (xy 144.665116 55.077416)
-					(xy 144.701387 55.148353) (xy 144.722382 55.228103)
+					(xy 144.380941 54.914311) (xy 144.465664 54.938006) (xy 144.541173 54.976637) (xy 144.608992 55.030857)
+					(xy 144.669972 55.102466) (xy 144.727032 55.20222) (xy 144.77072 55.325734) (xy 144.799221 55.477838)
+					(xy 144.809556 55.664194) (xy 144.799201 55.851678) (xy 144.770667 56.004445) (xy 144.726975 56.128257)
+					(xy 144.669972 56.228029) (xy 144.608997 56.2996) (xy 144.54118 56.353795) (xy 144.465671 56.392409)
+					(xy 144.380946 56.416095) (xy 144.284923 56.424309) (xy 144.188901 56.416096) (xy 144.104166 56.392412)
+					(xy 144.028637 56.353798) (xy 143.960792 56.299602) (xy 143.899782 56.228029) (xy 143.84282 56.128263)
+					(xy 143.799155 56.004454) (xy 143.770639 55.851684) (xy 143.760289 55.664194) (xy 144.079301 55.664194)
+					(xy 144.082039 55.770883) (xy 144.089742 55.863313) (xy 144.104282 55.949908) (xy 144.124364 56.018469)
+					(xy 144.153319 56.077837) (xy 144.187378 56.119036) (xy 144.230507 56.145509) (xy 144.284923 56.154665)
+					(xy 144.339507 56.145542) (xy 144.383475 56.119036) (xy 144.418173 56.077696) (xy 144.446489 56.018469)
+					(xy 144.4658 55.949963) (xy 144.480012 55.863313) (xy 144.487782 55.770882) (xy 144.490545 55.664194)
+					(xy 144.487773 55.55756) (xy 144.480012 55.466083) (xy 144.465823 55.380333) (xy 144.446489 55.312027)
+					(xy 144.418168 55.252721) (xy 144.383475 55.211368) (xy 144.339507 55.184862) (xy 144.284923 55.175739)
+					(xy 144.230507 55.184895) (xy 144.187378 55.211368) (xy 144.153324 55.25258) (xy 144.124364 55.312027)
+					(xy 144.104258 55.380389) (xy 144.089742 55.466083) (xy 144.082048 55.557559) (xy 144.079301 55.664194)
+					(xy 143.760289 55.664194) (xy 143.770026 55.487176) (xy 143.797017 55.340786) (xy 143.826239 55.248934)
+					(xy 143.861715 55.170368) (xy 143.902988 55.103474) (xy 143.953038 55.043309) (xy 144.008165 54.99465)
+					(xy 144.068768 54.95647) (xy 144.134765 54.928783) (xy 144.206434 54.91189) (xy 144.284923 54.906095)
 				)
 			)
